File: armduino.sch (EAGLE design)
At the start: 61 parts, among them IC1 78D2, IC3 LM1117-3.3V, Q1 12MHz, Q2 12MHz, T1 BC857, T2 BC857, U1 LPC11U35FBD48/401, U2 MKE02Z64VLD4, X1 POWERSUPPLY_DC21MMX, X2 USB-B_TH

Commit message: Version 0.4
Parts:
- removed C6: 100nF/25V, rcl:C-EUC0805K
- removed C7, C8: 33nF/25V, rcl:C-EUC0805K
- removed CONNECTED, RUNNING: (no value), led:LEDCHIP-LED0805
- removed Q1: 12MHz, crystal:CRYSTALSM49
- removed R11: 120r, rcl:R-EU_M0805
- removed T2: BC857, transistor:BC857A-PNP-SOT23-BEC
- removed U$1: SWITCH-4X4, pessoal:SWITCH-4X4
- removed U1: LPC11U35FBD48/401, NXP_By_element14_Batch_1:LPC11U35FBD48/401
- added C16, C19: 22pF, rcl:C-EUC0603K
- added C18: 2.2nF/16V, rcl:C-EUC0805K
- added C20: 1nF/25V, rcl:C-EUC0805K
- added CONNECTED1, RUNNING1: (no value), led:LEDCHIP-LED0805
- added Q3: 8MHz, crystal:CRYSTALHC49S
- added R20: 120r, rcl:R-EU_M0805
- added U3: MKL26ZVFM4, freescale:MKL26ZVFM4
- C5: value 100nF/25V -> 1nF/25V
- IC1: value 78D2 -> 7805DT; device linear:78D2 -> linear:7805DT
- R10: value 120r -> 20k
- R14: value 2.2k -> 1k
- R18: value 24k -> 4.7k
- R19: value 39k -> 10k
- R4: value 1.5k -> 10k
- R5: value 10k -> 1M
- R7: value 10k -> 20k
- R8: value 2.2k -> 120r
- T1: value BC857 -> S9012; device transistor:BC857A-PNP-SOT23-BEC -> transistor:-PNP-SOT23-BCE
Connections:
- removed net !USB_CON: R8.2, U1.PIO0_6/!USB_CONNECT!/SCK0
- removed net LPC_RESET: ICSP1.5, R9.2, U1.!RESET!/PIO0_0
- removed net LPC_SWCLK: ICSP1.1, U1.SWCLK/PIO0_10/SCK0/CT16B0_MAT2
- removed net LPC_SWDIO: ICSP1.3, U1.SWDIO/PIO0_15
- removed net N$10: C8.1, Q1.2, U1.XTALOUT
- removed net N$15: R10.1, RUNNING.C
- removed net N$16: CONNECTED.C, R11.1
- removed net N$9: C7.1, Q1.1, U1.XTALIN
- removed net PROG_SWO: U1.PIO1_25/CT32B0_MAT1
- removed net USB_VBUS: FUSE1.2, R18.1, T2.C
- new net DEBUG_RESET: ICSP1.5, R18.2, R19.1, U3.PTA20/RESET_B
- new net DEBUG_SWCLK: ICSP1.1, U3.PTA0/SWD_CLK/TSI0_CH1/TPM0_CH5
- new net DEBUG_SWDIO: ICSP1.3, U3.PTA3/SWD_DIO/TSI0_CH4/I2C1_SCL/TPM0_CH0
- new net N$12: CONNECTED1.C, R20.1
- new net N$25: C16.1, Q3.2, R5.1, U3.PTA19/XTAL0/UART1_TX/TPM_CLKIN1/LPTMR0_ALT1
- new net N$31: C18.1, U3.VOUT33
- new net USB_CON: FUSE1.2, R18.1, T1.E
- net +3V3: now also C20.1, U3.VDD, U3.VDDA; no longer C6.1, R5.1, R7.1, R9.1, T1.C, U1.VDD, U1.VDD@1
- net +5V: now also T1.C, U3.VREGIN; no longer T2.E
- net GND: now also C16.2, C18.2, C19.2, C20.2, R19.2, R20.2, R7.2, R8.2, U3.EXP, U3.VSS, U3.VSS@1, U3.VSSA; no longer C6.2, C7.2, C8.2, R11.2, R19.1, U$1G$1.P, U1.VSS, U1.VSS@1
- net N$11: now also RUNNING1.C; no longer R7.2, T1.B
- net N$13: now also RUNNING1.A, U3.PTC3/LLWU_P7/UART1_RX/TPM0_CH2/CLKOUT/I2S0_TX_BCLK; no longer RUNNING.A, U1.PIO0_22/AD6/CT16B1_MAT1/MISO1
- net N$14: now also CONNECTED1.A, U3.PTC1/LLWU_P6/RTC_CLKIN/ADC0_SE15/TSI0_CH14/I2C1_SCL/TPM0_CH0/I2S0_TXD0; no longer CONNECTED.A, U1.PIO0_23/AD7
- net N$22: now also T1.B; no longer T2.B
- net N$24: now also C19.1, Q3.1, R5.2, U3.PTA18/EXTAL0/UART1_RX/TPM_CLKIN0; no longer R18.2, R19.2, U1.PIO0_3/USB_VBUS
- net N$6: now also R10.1, R9.2, U3.PTD6/LLWU_P15/ADC0_SE7B/SPI1_MOSI/UART0_RX/SPI1_MISO; no longer R5.2, U$1G$1.S, U1.PIO0_1/CLKOUT/CT32B0_MAT2/USB_FTOGGLE
- net N$8: now also R4.2, R7.1, U3.PTC6/LLWU_P10/CMP0_IN0/SPI0_MOSI/EXTRG_IN/I2S0_RX_BCLK/SPI0_MISO/I2S0_MCLK; no longer R4.1, T1.E
- net PROG_NRESET: now also U3.PTD5/ADC0_SE6B/SPI1_SCK/UART2_TX/TPM0_CH5; no longer U1.PIO1_27/CT32B0_MAT3/TXD
- net PROG_RX: now also R9.1; no longer U1.PIO0_18/RXD/CT32B0_MAT0
- net PROG_SWCLK: now also U3.PTC5/LLWU_P9/SPI0_SCK/LPTMR0_ALT2/I2S0_RXD0/CMP0_OUT; no longer U1.PIO1_19/!DTR!/SSEL1
- net PROG_SWDIO: now also R4.1, U3.PTC7/CMP0_IN1/SPI0_MISO/AUDIOUSB_SOF_OUT/I2S0_RX_FS/SPI0_MOSI; no longer U1.PIO1_20/!DSR!/SCK1
- net PROG_TX: now also U3.PTD7/SPI1_MISO/UART0_TX/SPI1_MOSI; no longer U1.PIO0_19/TXD/CT32B0_MAT1
- net USB_D+: now also U3.USB0_DP; no longer R4.2, U1.USB_DP
- net USB_D-: now also U3.USB0_DM; no longer U1.USB_DM
Other:
- moved on the sheet: C5, ICSP1, R10, R18, R19, R4, R5, R7, R8, R9, T1

Commit message: Removed PWM 3 and 5 from FTM0_FLT pins.
Some pins were moved around to fit PWM on FTM_CHx pins.
Parts:
- removed T1: S9012, transistor:-PNP-SOT23-BCE
- added T2: BC846, transistor:BC857A-PNP-SOT23-BEC
- R14: value 1k -> 2.2k
Connections:
- net +5V: now also T2.E; no longer T1.C
- net N$22: now also T2.B; no longer T1.B
- net UC_IO_2: now also U2.PTA7/FTM2_FLT2/ACMP1_IN1/ADC0_SE3; no longer U2.PTD4/KBI1_P4
- net UC_IO_4: now also U2.PTA6/FTM2_FLT1/ACMP1_IN0/ADC0_SE2; no longer U2.PTD7/KBI1_P7/UART2_TX
- net UC_IO_7: now also U2.PTD4/KBI1_P4; no longer U2.PTD6/KBI1_P6/UART2_RX
- net UC_PWM_3: now also U2.PTB5/FTM2_CH5/SPI0_PCS0/ACMP1_OUT; no longer U2.PTA7/FTM2_FLT2/ACMP1_IN1/ADC0_SE3
- net UC_PWM_5: now also U2.PTH2/BUSOUT/FTM1_CH0; no longer U2.PTA6/FTM2_FLT1/ACMP1_IN0/ADC0_SE2
- net UC_PWM_6: now also U2.PTE7/FTM2_CLK/FTM1_CH1; no longer U2.PTB5/FTM2_CH5/SPI0_PCS0/ACMP1_OUT
- net USB_CON: now also T2.C; no longer T1.E
Changed lines of the file:
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@@
 <layers>
 <layer number="1" name="Top" color="4" fill="1" visible="no" active="no"/>
-<layer number="2" name="Route2" color="1" fill="3" visible="no" active="no"/>
-<layer number="3" name="Route3" color="4" fill="3" visible="no" active="no"/>
-<layer number="4" name="Route4" color="1" fill="4" visible="no" active="no"/>
-<layer number="5" name="Route5" color="4" fill="4" visible="no" active="no"/>
-<layer number="6" name="Route6" color="1" fill="8" visible="no" active="no"/>
-<layer number="7" name="Route7" color="4" fill="8" visible="no" active="no"/>
-<layer number="8" name="Route8" color="1" fill="2" visible="no" active="no"/>
-<layer number="9" name="Route9" color="4" fill="2" visible="no" active="no"/>
-<layer number="10" name="Route10" color="1" fill="7" visible="no" active="no"/>
-<layer number="11" name="Route11" color="4" fill="7" visible="no" active="no"/>
-<layer number="12" name="Route12" color="1" fill="5" visible="no" active="no"/>
-<layer number="13" name="Route13" color="4" fill="5" visible="no" active="no"/>
-<layer number="14" name="Route14" color="1" fill="6" visible="no" active="no"/>
-<layer number="15" name="Route15" color="4" fill="6" visible="no" active="no"/>
 <layer number="16" name="Bottom" color="1" fill="1" visible="no" active="no"/>
 <layer number="17" name="Pads" color="2" fill="1" visible="no" active="no"/>
@@
 <part name="+3V7" library="supply1" deviceset="+3V3" device=""/>
 <part name="Q2" library="crystal" deviceset="CRYSTAL" device="SM49" value="12MHz"/>
-<part name="R14" library="rcl" deviceset="R-EU_" device="M0805" value="1k"/>
+<part name="T2" library="transistor" deviceset="*-PNP-" device="SOT23-BEC" technology="BC857A" value="BC846"/>
+<part name="R14" library="rcl" deviceset="R-EU_" device="M0805" value="2.2k"/>
 <part name="P+10" library="supply1" deviceset="VCC" device=""/>
 <part name="U3" library="freescale" deviceset="MKL26Z*VFM4" device=""/>
@@
 <part name="R10" library="rcl" deviceset="R-EU_" device="M0805" value="20k"/>
 <part name="GND7" library="supply1" deviceset="GND" device=""/>
-<part name="T1" library="transistor" deviceset="*-PNP-" device="SOT23-BCE" value="S9012"/>
 </parts>
 <sheets>
@@
 <instance part="+3V7" gate="G$1" x="-5.08" y="180.34"/>
 <instance part="Q2" gate="G$1" x="81.28" y="144.78"/>
+<instance part="T2" gate="G$1" x="-139.7" y="187.96"/>
 <instance part="R14" gate="G$1" x="-149.86" y="187.96"/>
 <instance part="P+10" gate="VCC" x="-157.48" y="208.28"/>
@@
 <instance part="R10" gate="G$1" x="48.26" y="96.52" rot="R270"/>
 <instance part="GND7" gate="1" x="48.26" y="0"/>
-<instance part="T1" gate="G$1" x="-139.7" y="187.96" rot="MR180"/>
 </instances>
 <busses>
@@
 </segment>
 <segment>
+<pinref part="T2" gate="G$1" pin="E"/>
 <pinref part="P+5" gate="1" pin="+5V"/>
 <wire x1="-137.16" y1="193.04" x2="-137.16" y2="205.74" width="0.1524" layer="91"/>
-<pinref part="T1" gate="G$1" pin="C"/>
 </segment>
 <segment>
@@
 </segment>
 <segment>
+<pinref part="U2" gate="G$1" pin="PTE7/FTM2_CLK/FTM1_CH1"/>
+<wire x1="144.78" y1="106.68" x2="142.24" y2="106.68" width="0.1524" layer="91"/>
+<label x="142.24" y="106.68" size="1.016" layer="95" font="vector" ratio="7" rot="R180" xref="yes"/>
+</segment>
+</net>
+<net name="UC_PWM_3" class="0">
+<segment>
+<pinref part="IOL" gate="A" pin="4"/>
+<wire x1="332.74" y1="78.74" x2="325.12" y2="78.74" width="0.1524" layer="91"/>
+<label x="325.12" y="78.74" size="1.016" layer="95" font="vector" rot="R180" xref="yes"/>
+</segment>
+<segment>
 <pinref part="U2" gate="G$1" pin="PTB5/FTM2_CH5/SPI0_PCS0/ACMP1_OUT"/>
 <wire x1="144.78" y1="96.52" x2="142.24" y2="96.52" width="0.1524" layer="91"/>
@@
 </segment>
 </net>
-<net name="UC_PWM_3" class="0">
-<segment>
-<pinref part="IOL" gate="A" pin="4"/>
-<wire x1="332.74" y1="78.74" x2="325.12" y2="78.74" width="0.1524" layer="91"/>
-<label x="325.12" y="78.74" size="1.016" layer="95" font="vector" rot="R180" xref="yes"/>
-</segment>
-<segment>
-<pinref part="U2" gate="G$1" pin="PTA7/FTM2_FLT2/ACMP1_IN1/ADC0_SE3"/>
-<wire x1="264.16" y1="93.98" x2="266.7" y2="93.98" width="0.1524" layer="91"/>
-<label x="266.7" y="93.98" size="1.016" layer="95" font="vector" xref="yes"/>
-</segment>
-</net>
 <net name="UC_PWM_5" class="0">
 <segment>
@@
 </segment>
 <segment>
-<pinref part="U2" gate="G$1" pin="PTA6/FTM2_FLT1/ACMP1_IN0/ADC0_SE2"/>
-<wire x1="264.16" y1="99.06" x2="266.7" y2="99.06" width="0.1524" layer="91"/>
-<label x="266.7" y="99.06" size="1.016" layer="95" font="vector" xref="yes"/>
+<pinref part="U2" gate="G$1" pin="PTH2/BUSOUT/FTM1_CH0"/>
+<wire x1="144.78" y1="101.6" x2="142.24" y2="101.6" width="0.1524" layer="91"/>
+<label x="142.24" y="101.6" size="1.016" layer="95" font="vector" ratio="7" rot="R180" xref="yes"/>
 </segment>
 </net>
@@
 </segment>
 <segment>
-<pinref part="U2" gate="G$1" pin="PTD7/KBI1_P7/UART2_TX"/>
-<wire x1="144.78" y1="76.2" x2="142.24" y2="76.2" width="0.1524" layer="91"/>
-<label x="142.24" y="76.2" size="1.016" layer="95" font="vector" rot="R180" xref="yes"/>
+<pinref part="U2" gate="G$1" pin="PTA6/FTM2_FLT1/ACMP1_IN0/ADC0_SE2"/>
+<wire x1="264.16" y1="99.06" x2="266.7" y2="99.06" width="0.1524" layer="91"/>
+<label x="266.7" y="99.06" size="1.016" layer="95" font="vector" ratio="7" xref="yes"/>
 </segment>
 </net>
@@
 </segment>
 <segment>
-<pinref part="U2" gate="G$1" pin="PTD4/KBI1_P4"/>
-<wire x1="264.16" y1="104.14" x2="266.7" y2="104.14" width="0.1524" layer="91"/>
-<label x="266.7" y="104.14" size="1.016" layer="95" font="vector" xref="yes"/>
+<pinref part="U2" gate="G$1" pin="PTA7/FTM2_FLT2/ACMP1_IN1/ADC0_SE3"/>
+<wire x1="264.16" y1="93.98" x2="266.7" y2="93.98" width="0.1524" layer="91"/>
+<label x="266.7" y="93.98" size="1.016" layer="95" font="vector" ratio="7" xref="yes"/>
 </segment>
 </net>
@@
 </segment>
 <segment>
-<pinref part="U2" gate="G$1" pin="PTD6/KBI1_P6/UART2_RX"/>
-<wire x1="144.78" y1="71.12" x2="142.24" y2="71.12" width="0.1524" layer="91"/>
-<label x="142.24" y="71.12" size="1.016" layer="95" font="vector" rot="R180" xref="yes"/>
+<pinref part="U2" gate="G$1" pin="PTD4/KBI1_P4"/>
+<wire x1="264.16" y1="104.14" x2="266.7" y2="104.14" width="0.1524" layer="91"/>
+<label x="266.7" y="104.14" size="1.016" layer="95" font="vector" ratio="7" xref="yes"/>
 </segment>
 </net>
@@
 <pinref part="FUSE1" gate="G$1" pin="2"/>
 <wire x1="-139.7" y1="167.64" x2="-137.16" y2="167.64" width="0.1524" layer="91"/>
+<pinref part="T2" gate="G$1" pin="C"/>
 <wire x1="-137.16" y1="167.64" x2="-137.16" y2="177.8" width="0.1524" layer="91"/>
 <wire x1="-137.16" y1="177.8" x2="-137.16" y2="182.88" width="0.1524" layer="91"/>
@@
 <junction x="-137.16" y="177.8"/>
 <label x="-142.24" y="177.8" size="1.016" layer="95" font="vector" rot="R180" xref="yes"/>
-<pinref part="T1" gate="G$1" pin="E"/>
 </segment>
 <segment>
@@
 <segment>
 <pinref part="R14" gate="G$1" pin="2"/>
+<pinref part="T2" gate="G$1" pin="B"/>
 <wire x1="-144.78" y1="187.96" x2="-142.24" y2="187.96" width="0.1524" layer="91"/>
-<pinref part="T1" gate="G$1" pin="B"/>
-</segment>
-</net>
+</segment>
+</net>

Commit message: Correct voltage source selection, correct target XTAL.
 * Add LM358 to switch between external connector and USB source;
 * Target using 20MHz external crystal;
 * Re-route to fit new components;
Parts:
- removed RESET: SWITCH-4X4, pessoal:SWITCH-4X4
- removed T2: BC846, transistor:BC857A-PNP-SOT23-BEC
- added C6: 100nF/50V, rcl:C-EUC0805K
- added IC2: LM358D, linear:LM358D
- added Q1: FDN360P, transistor-power:FDN360P
- added R11: 10k, rcl:R-EU_M0805
- added S1: (no value), switch-omron:10-XX
- C3, C4: value 10uF/35V -> 10uF/16V; device rcl:CPOL-EU153CLV-0505 -> rcl:CPOL-EUE2-4
- D1: device diode:DIODE-DO214AC -> diode:DIODE-DO-214AC
- Q2: value 12MHz -> 20MHz
- R14: value 2.2k -> 10k
- renumbered CONNECTED1 to CONN, LED2 to USB, RUNNING1 to RUN
Connections:
- net N$12 renamed CONN
- removed net N$22: R14.2, T2.B
- new net N$15: IC2A.+IN, R11.1, R14.2
- new net N$26: IC2A.OUT, Q1.G
- new net N$9: C3.+, IC3.IN
- net +3V3: now also IC2A.-IN
- net +5V: now also C6.1, IC2P.V+, Q1.S; no longer C3.+, IC3.IN, T2.E
- net GND: now also C6.2, IC2B.+IN, IC2B.-IN, IC2P.V-, R14.1, S1.P; no longer RESETG$1.P, X2.P$1, X2.P$2
- net PROG_NRESET: now also S1.S; no longer RESETG$1.S
- net USB_CON: now also Q1.D; no longer T2.C
- net VCC: now also R11.2; no longer R14.1
Other:
- note added: "USE TANTALUM CAPACITORS FOR C3 AND C4"
- moved on the sheet: C1, C2, D1, IC1, R14, X1

Commit message: Modifications to v0.7:  * Schematic parts grouped together;  * KL26 footprint edited with extended pads, for easier soldering;  * SWD signal rerouting to avoid transpositions and unnecessary curves;  * Added SWD connection for external target;  * Corrected Programmer name.
Parts:
- removed U3: MKL26ZVFM4, freescale:MKL26ZVFM4
- added ICSP2: 3x2 M, SmartPrj:PINHD-2X3
- added U1: MKL26Z128VFM4, freescale:MKL26Z128VFM4
Connections:
- removed net N$14: CONN.A, U3.PTC1/LLWU_P6/RTC_CLKIN/ADC0_SE15/TSI0_CH14/I2C1_SCL/TPM0_CH0/I2S0_TXD0
- removed net N$31: C18.1, U3.VOUT33
- new net N$10: C18.1, U1.VOUT33
- new net N$12: RUN.A, U1.PTC3/LLWU_P7
- net +3V3: now also U1.VDD, U1.VDDA; no longer U3.VDD, U3.VDDA
- net +5V: now also ICSP2.2, U1.VREGIN; no longer U3.VREGIN
- net DEBUG_RESET: now also U1.PTA20; no longer U3.PTA20/RESET_B
- net DEBUG_SWCLK: now also U1.PTA0; no longer U3.PTA0/SWD_CLK/TSI0_CH1/TPM0_CH5
- net DEBUG_SWDIO: now also U1.PTA3; no longer U3.PTA3/SWD_DIO/TSI0_CH4/I2C1_SCL/TPM0_CH0
- net GND: now also ICSP2.6, U1.EPAD, U1.VSS, U1.VSSA, U1.VSS_2; no longer U3.EXP, U3.VSS, U3.VSS@1, U3.VSSA
- net N$13: now also CONN.A, U1.PTC1/LLWU_P6/RTC_CLKIN; no longer RUN.A, U3.PTC3/LLWU_P7/UART1_RX/TPM0_CH2/CLKOUT/I2S0_TX_BCLK
- net N$24: now also U1.PTA18; no longer U3.PTA18/EXTAL0/UART1_RX/TPM_CLKIN0
- net N$25: now also U1.PTA19; no longer U3.PTA19/XTAL0/UART1_TX/TPM_CLKIN1/LPTMR0_ALT1
- net N$6: now also U1.PTD6/LLWU_P15; no longer U3.PTD6/LLWU_P15/ADC0_SE7B/SPI1_MOSI/UART0_RX/SPI1_MISO
- net N$8: now also U1.PTC6/LLWU_P10; no longer U3.PTC6/LLWU_P10/CMP0_IN0/SPI0_MOSI/EXTRG_IN/I2S0_RX_BCLK/SPI0_MISO/I2S0_MCLK
- net PROG_NRESET: now also ICSP2.5, U1.PTD5; no longer U3.PTD5/ADC0_SE6B/SPI1_SCK/UART2_TX/TPM0_CH5
- net PROG_SWCLK: now also ICSP2.1, U1.PTC5/LLWU_P9; no longer U3.PTC5/LLWU_P9/SPI0_SCK/LPTMR0_ALT2/I2S0_RXD0/CMP0_OUT
- net PROG_SWDIO: now also ICSP2.3, U1.PTC7; no longer U3.PTC7/CMP0_IN1/SPI0_MISO/AUDIOUSB_SOF_OUT/I2S0_RX_FS/SPI0_MOSI
- net PROG_TX: now also U1.PTD7; no longer U3.PTD7/SPI1_MISO/UART0_TX/SPI1_MOSI
- net USB_D+: now also U1.USB0_DP; no longer U3.USB0_DP
- net USB_D-: now also U1.USB0_DM; no longer U3.USB0_DM
Other:
- note added: "PINOUT"
- note added: "POWER"
- note added: "PROGRAMMER/DEBUGGER"
- note added: "TARGET"
- moved on the sheet: AD, C1, C10, C11, C12, C13, C14, C15, C16, C17, C18, C19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

Commit message: Add led values according to colors to be used and fuse value.
Parts:
- Q2: value 20MHz -> 5MHz
Changed lines of the file:
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@@
 <part name="GND29" library="supply1" deviceset="GND" device=""/>
 <part name="+3V7" library="supply1" deviceset="+3V3" device=""/>
-<part name="Q2" library="crystal" deviceset="CRYSTAL" device="SM49" value="20MHz"/>
+<part name="Q2" library="crystal" deviceset="CRYSTAL" device="SM49" value="5MHz"/>
 <part name="Q3" library="crystal" deviceset="CRYSTAL" device="HC49S" value="8MHz"/>
 <part name="GND24" library="supply1" deviceset="GND" device=""/>
